File: hardware/oven_rev3/oven_rev3.kicad_sch (KiCad schematic)
At the start: 22 parts, among them J1 RELAY_CTRL, J10 5V_IN, J2 SERIAL, J3 NUMPAD, J4 AVR-ISP-6, J5 LIVE, J6 DISPLAY, J7 RELAY_PWR, J8 OUTPUT, J9 NEUTRAL, U1 ATmega328-AU, U2 MAX6675, Y1 16M

Commit message: Touched up title blocks and rev 3
Connections:
- net GND: no longer J8.1 (Pin_1), U2.2 (T-)
- new net TC-: J8.1 (Pin_1), U2.2 (T-)
